File: accl.kicad_sch (KiCad schematic)
At the start: 2 parts, among them U5 ADXL343

Commit message: Final refinements before issue to JLC
Parts:
- renumbered C16 to C19, U5 to U6
Changed lines of the file:
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@@
   (symbol (lib_id "power:+3V3") (at 57.15 25.4 0) (unit 1)
     (in_bom yes) (on_board yes) (fields_autoplaced)
-    (property "Reference" "#PWR039" (id 0) (at 57.15 29.21 0)
+    (property "Reference" "#PWR041" (id 0) (at 57.15 29.21 0)
       (effects (font (size 1.27 1.27)) hide)
     )
@@
   (symbol (lib_id "Sensor_Motion:ADXL343") (at 52.07 45.72 0) (unit 1)
     (in_bom yes) (on_board yes) (fields_autoplaced)
-    (property "Reference" "U5" (id 0) (at 67.31 39.1412 0))
+    (property "Reference" "U6" (id 0) (at 67.31 39.1412 0))
     (property "Value" "ADXL343" (id 1) (at 67.31 41.6812 0))
     (property "Footprint" "Package_LGA:LGA-14_3x5mm_P0.8mm_LayoutBorder1x6y" (id 2) (at 52.07 45.72 0)
@@
   (symbol (lib_id "Device:C_Small") (at 88.9 35.56 0) (unit 1)
     (in_bom yes) (on_board yes) (fields_autoplaced)
-    (property "Reference" "C16" (id 0) (at 91.44 34.2962 0)
+    (property "Reference" "C19" (id 0) (at 91.44 34.2962 0)
       (effects (font (size 1.27 1.27)) (justify left))
     )
@@
   (symbol (lib_id "power:GND") (at 52.07 63.5 0) (unit 1)
     (in_bom yes) (on_board yes) (fields_autoplaced)
-    (property "Reference" "#PWR038" (id 0) (at 52.07 69.85 0)
+    (property "Reference" "#PWR040" (id 0) (at 52.07 69.85 0)
       (effects (font (size 1.27 1.27)) hide)
     )
@@
   (symbol (lib_id "power:+3V3") (at 88.9 24.13 0) (unit 1)
     (in_bom yes) (on_board yes) (fields_autoplaced)
-    (property "Reference" "#PWR040" (id 0) (at 88.9 27.94 0)
+    (property "Reference" "#PWR042" (id 0) (at 88.9 27.94 0)
       (effects (font (size 1.27 1.27)) hide)
     )
@@
   (symbol (lib_id "power:GND") (at 88.9 46.99 0) (unit 1)
     (in_bom yes) (on_board yes) (fields_autoplaced)
-    (property "Reference" "#PWR041" (id 0) (at 88.9 53.34 0)
+    (property "Reference" "#PWR043" (id 0) (at 88.9 53.34 0)
       (effects (font (size 1.27 1.27)) hide)
     )
